File: Serialdac-dff.kicad_sch (KiCad schematic)
At the start: 59 parts

Commit message: V1.1
Parts:
- added J5: Conn_01x03_Pin, Connector_PinHeader_2.54mm:PinHeader_1x03_P2.54mm_Vertical, symbol Connector:Conn_01x03_Pin
- gave numbers to parts that had none: 59
Connections:
- net GNDA: now also J5.2 (Pin_2)
- net VDD: now also J5.1 (Pin_1)
- net VEE: now also J5.3 (Pin_3)
