File: Serialdac.kicad_sch (KiCad schematic)
At the start: 53 parts, among them J5 Conn_01x03_Pin, J8 RJ-2410N, J9 RJ-2410N, K1 UD2-5NUN, Q1 2SA1162-GR, Q2 2SA1162-GR, Q3 BSS138, Q6 BSS138, U16 DAC8811IBDGKT, U17 DAC8811IBDGKT, U2 MAU106, U23 OPA2277, U24 OPA2277, U3 Si5351A-B-GT, U4 TL431PK, Y2 FA-238_25.0000MB-K3

Commit message: V2.0
Parts:
- removed K1: UD2-5NUN, pretty:UD25NUN, symbol xSSDAC:UD2-5NUN
- added C37, C40: 100n, Capacitor_SMD:C_0603_1608Metric_Pad1.08x0.95mm_HandSolder, symbol Device:C_Small
- added K1: UD2-5NU, SamacSys:UD25NUN, symbol SamacSys_Parts:UD2-5NU
- added TP33: TestPoint, pretty:TestPoint_Pad_3.0x3.0mm, symbol Connector:TestPoint
- C52, C53: value 16SEPC100M -> OS-CON 16SEPC100M; Akizuki Price/Stock (none) -> https://akizukidenshi.com/catalog/g/gP-08290/; Manufacturer_Name (none) -> Panasonic; Manufacturer_Part_Number (none) -> OS-CON 16SEPC100M
- C54: value 16MU106MC44532 -> PLMCAP 10uF 16V
- D1: value LED -> LED(Red); Manufacturer_Name (none) -> OptSupply; Manufacturer_Part_Number (none) -> OSHR1608C1A
- J5: value Conn_01x03_Pin -> PIN HEADER 01x03
- J8, J9: value RJ-2410N -> RCA JACK RJ-2410N
- NT1: value NetTie_2 -> Net-tie, cupper only
- Q3: Manufacturer_Name (none) -> BSS138; Manufacturer_Part_Number (none) -> BSS138
- Q4: renamed from Q6; Manufacturer_Name (none) -> BSS138; Manufacturer_Part_Number (none) -> BSS138
- R43, R44, R45, R46, R61, R62, R63, R64: footprint Resistor_SMD:R_0603_1608Metric_Pad0.98x0.95mm_HandSolder -> Resistor_THT:R_Axial_DIN0204_L3.6mm_D1.6mm_P2.54mm_Vertical
- U23, U24: value OPA2277 -> OPA2277UA; Manufacturer_Name (none) -> Texas Instruments; Manufacturer_Part_Number (none) -> OPA2277UA
- U3: Manufacturer_Name (none) -> Silicon Laboratories; Manufacturer_Part_Number (none) -> Si5351A-B-GT
- U4: Manufacturer_Name (none) -> Toshiba; Manufacturer_Part_Number (none) -> TA76431F
- renumbered R42 to R39
Connections:
- net +3V3: now also C37.2, C40.2
- net +5V: now also K1.1 (COIL_+)
- net GND: now also C37.1, C40.1
- net GNDA: now also K1.3 (COM_1), K1.6 (COM_2)
- net OUT_L: now also K1.7 (NC_2)
- net OUT_R: now also K1.2 (NC_1)
- net VREF: now also TP33.1
- net at D5.2, Q3.3 (D): now also K1.8 (COIL_-)
Other:
- note added: "RF return path"
- moved on the sheet: C46, C52, C53, C54, C55, C57, C59, C61, C64, D1, D5, J5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
