File: UnusedPin.kicad_sch (KiCad schematic)
At the start: 31 parts

Commit message: V1.1
Parts:
- gave numbers to parts that had none: 31

Commit message: V2.0
Parts:
- removed TP39, TP40, TP51: TestPoint, pretty:TestPoint_Pad_D1.0mm_noCrtYd, symbol Connector:TestPoint
- added TP32, TP33, TP4: TestPoint, pretty:TestPoint_Pad_3.0x3.0mm, symbol Connector:TestPoint
- added TP34, TP35, TP36: TestPoint, pretty:TestPoint_Pad_D1.0mm_noCrtYd, symbol Connector:TestPoint
- TP27, TP28, TP30: footprint TestPoint:TestPoint_Pad_4.0x4.0mm -> pretty:TestPoint_Pad_3.0x3.0mm
Connections:
- new net +1V0: TP33.1
- new net +3V3: TP32.1
- new net +5V: TP4.1
- new net X0D24: TP34.1
- new net X1D0: TP35.1
- new net X1D1: TP36.1
- no-connect marks 16 -> 11
Other:
- note added: "Port X1D14 - X1D21 unavailable if RGMII or USB enabled on tile 1 / tile 3 (as appropriate)"
- note added: "Port X1D2 - X1D9 unavailable if USB enabled on that tile"
- moved on the sheet: TP15, TP16, TP17, TP18, TP19, TP20, TP21, TP22, TP23, TP24, TP25, TP26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
