File: xCORE.kicad_sch (KiCad schematic)
At the start: 96 parts

Commit message: V1.1
Parts:
- removed ?: SJPA-D3, pretty:D_SJP_Handsoldering, symbol Device:D_Schottky
- added J7: Conn_01x02_Pin, Connector_PinHeader_2.54mm:PinHeader_1x02_P2.54mm_Vertical, symbol Connector:Conn_01x02_Pin
- added R60: 10K, Resistor_SMD:R_0603_1608Metric_Pad0.98x0.95mm_HandSolder, symbol Device:R_Small_US
- U5: renamed from ?; footprint SOTFL50P160X60-5N -> pretty:SOTFL50P160X60-5N
- gave numbers to parts that had none: 94
Connections:
- net +3V3: now also R60.1
- net +5V: now also J7.2 (Pin_2)
- net X0D1: now also U6.1 (CE#); no longer U6.2 (IO1)
- net X0D5: now also U6.2 (IO1), R60.2; no longer U6.1 (CE#)
- net at C2.1, FB1.1, R59.2: now also J7.1 (Pin_1)
- no-connect marks 25 -> 10

Commit message: V2.0
Parts:
- removed C10: 4.7u (0805), Capacitor_SMD:C_0805_2012Metric_Pad1.18x1.45mm_HandSolder, symbol Device:C_Small
- removed C13: 8p, Capacitor_SMD:C_0603_1608Metric_Pad1.08x0.95mm_HandSolder, symbol Device:C_Small
- removed C18: 1n, Capacitor_SMD:C_0603_1608Metric_Pad1.08x0.95mm_HandSolder, symbol Device:C_Small
- removed C21, C22, C35, C37: 100n, Capacitor_SMD:C_0603_1608Metric_Pad1.08x0.95mm_HandSolder, symbol Device:C_Small
- removed C40: 560p, Capacitor_SMD:C_0603_1608Metric_Pad1.08x0.95mm_HandSolder, symbol Device:C_Small
- removed C41: 2.7n, Capacitor_SMD:C_0603_1608Metric_Pad1.08x0.95mm_HandSolder, symbol Device:C_Small
- removed C43: 22u (1206), Capacitor_SMD:C_1206_3216Metric_Pad1.33x1.80mm_HandSolder, symbol Device:C_Small
- removed D2, D3: SJPA-D3, pretty:D_SJP_Handsoldering, symbol Device:D_Schottky
- removed J3: 625-7296, SamacSys_Parts:SHDR20W64P254_2X10_3305X860X930P, symbol xSSDAC-rescue:625-7296-SamacSys_Parts
- removed L1: NR6028T100M, SamacSys_Parts:NR6020T2R2N, symbol xSSDAC:NR10050T4R9N
- removed R12: 62K, Resistor_SMD:R_0603_1608Metric_Pad0.98x0.95mm_HandSolder, symbol Device:R_Small_US
- removed R14: 100K, Resistor_SMD:R_0603_1608Metric_Pad0.98x0.95mm_HandSolder, symbol Device:R_Small_US
- removed R17: 71.5k, Resistor_SMD:R_0603_1608Metric_Pad0.98x0.95mm_HandSolder, symbol Device:R_Small_US
- removed R19: 120K, Resistor_SMD:R_0603_1608Metric_Pad0.98x0.95mm_HandSolder, symbol Device:R_Small_US
- removed R21: 6.3k, Resistor_SMD:R_0603_1608Metric_Pad0.98x0.95mm_HandSolder, symbol Device:R_Small_US
- removed R22: 80.6k, Resistor_SMD:R_0603_1608Metric_Pad0.98x0.95mm_HandSolder, symbol Device:R_Small_US
- removed R23: 10.2k, Resistor_SMD:R_0603_1608Metric_Pad0.98x0.95mm_HandSolder, symbol Device:R_Small_US
- removed R24: 20k, Resistor_SMD:R_0603_1608Metric_Pad0.98x0.95mm_HandSolder, symbol Device:R_Small_US
- removed R25: 0, Resistor_SMD:R_0603_1608Metric_Pad0.98x0.95mm_HandSolder, symbol Device:R_Small_US
- removed R26: 20K, Resistor_SMD:R_0603_1608Metric_Pad0.98x0.95mm_HandSolder, symbol Device:R_Small_US
- removed U18: TAR5S25U(F), TO_SOT_Packages_SMD:SOT-23-5, symbol xSSDAC:TAR5S25U(F)-TAR5S25U(F)
- removed U19, U20: MP1584EN-LF-Z, pretty:SOIC127P600X170-9N, symbol xSSDAC:MP1584EN-LF-Z
- removed U6: IS25LP080D-JBLE, pretty:SOIC127P600X175-8N, symbol xSSDAC:IS25LP080D-JBLE-IS25LP080D-JBLE
- added C11: 100n, Capacitor_SMD:C_0603_1608Metric_Pad1.08x0.95mm_HandSolder, symbol Device:C_Small
- added J3: BOX HEADER 02x10, SamacSys:SHDRRA20W66P254_2X10_3289X986X927P, symbol SamacSys_Parts:5103310-5
- added TP34: TestPoint, pretty:TestPoint_Pad_D1.0mm_noCrtYd, symbol Connector:TestPoint
- added U10: NJM12877F33-TE1, Package_TO_SOT_SMD:SOT-23-5_HandSoldering, symbol SamacSys_Parts:NJM12877F33-TE1
- added U11: MPQ2172GJ-AEC1-Z, pretty:MPQ2172GJAEC1Z, symbol SamacSys_Parts:MPQ2172GJ-AEC1-Z
- added U18: NJM12877F25-TE1, Package_TO_SOT_SMD:SOT-23-5_HandSoldering, symbol SamacSys_Parts:NJM12877F33-TE1
- added U6: S25FL132K0XMFI013, SamacSys:SOIC127P800X216-8N, symbol SamacSys_Parts:S25FL132K0XMFI013
- C12: value 2p -> 330n
- C13: renamed from C44; value 33u (1206) -> 22u (1206)
- C17: value 560p -> 10n
- C5: value 10n -> 100n
- C7: value 1u -> 220n
- C8: value 10u (0805) -> 10n; footprint Capacitor_SMD:C_0805_2012Metric_Pad1.18x1.45mm_HandSolder -> Capacitor_SMD:C_0603_1608Metric_Pad1.08x0.95mm_HandSolder
- J2: value ZX62-B-5PA_11 -> USB JACK ZX62-B-5PA_11
- J7: value Conn_01x02_Pin -> PIN HEADER 01x02
- L1: renamed from L2; value NR6028T4R7N -> 0.47uH, 8.7A (1210); footprint SamacSys_Parts:NR6020T2R2N -> Inductor_SMD:L_1210_3225Metric_Pad1.42x2.65mm_HandSolder; Manufacturer_Name TAIYO YUDEN -> MURATA MFG.CO., LTD; Manufacturer_Part_Number NR10050T4R9N -> DFE32CAHR47MR0
- R13: value 22k -> 100K
- R14: renamed from R18; value 71.5k -> 24K
- R15: renamed from R20; value 160k -> 36K
- U1: footprint pretty:QFP40P1600X1600X120-129N-D-TH -> pretty:QFP40P1600X1600X120-129N-D
- Y1: Manufacturer_Name (none) -> CITIZEN; Manufacturer_Part_Number (none) -> HC49/U-S24000000ABJB
- renumbered C11 to C10, R15 to R12, S1 to SW8
Connections:
- net +1V0: now also R14.1, U11.5 (OUT)
- net +2V5: now also C7.1, U18.5 (VOUT); no longer C8.1
- net +3V3: now also C12.1, C36.2, U10.5 (VOUT), U6.8 (VCC)
- net +5V: now also C5.1, C11.1, U10.1 (VIN), U10.3 (CONTROL), U11.2 (VIN), U18.1 (VIN), U18.3 (CONTROL); no longer C7.1
- net GND: now also C36.1, R13.1, C11.2, J3.1, J3.13, J3.17, J3.5, J3.9, U10.2 (GND), U11.4 (PGND), U11.6 (AGND), U18.2 (GND), U6.4 (VSS); no longer R14.2
- net X0D1: now also U6.1 (CS#)
- net X0D10: now also U6.6 (SCK)
- net X0D4: now also U6.5 (SI/IO0)
- net X0D40: now also J3.3
- net X0D41: now also J3.7
- net X0D5: now also U6.2 (SO/IO1)
- net X0D6: now also U6.3 (WP#/IO2)
- net X0D7: now also U6.7 (HOLD#/IO3)
- net at L1.1: now also U11.3 (SW)
- net at R12.2: now also R13.2, U11.8 (EN); no longer R14.1
- net at R15.2: now also R14.2, U11.7 (FB)
- net at R8.2, U9.3 (A2): now also J3.6
- net at R6.1: now also J3.15
- net at R5.1: now also J3.11
- net at U1.1 (TDO): now also J3.8
- net at U1.127 (TMS): now also J3.14
- net at U1.128 (TCK): now also J3.12
- net at U1.2 (TDI): now also J3.16
- net at C17.1: now also U10.4 (CS)
- new net: TP34.1, U11.1 (PG)
- new net: C8.1, U18.4 (CS)
Other:
- note added: "--> 0"
- moved on the sheet: C10, C13, C16, C25, C32, L1, R12, R13, R14, R15, R16, R51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
