File: xSSDAC.kicad_sch (KiCad schematic)
At the start: 8 parts

Commit message: V1.1
Parts:
- gave numbers to parts that had none: 8
Other:
- company: (none) -> xken
- title: (none) -> xSSDAC SD player v1.1 

Commit message: V2.0
Parts:
- added ART1: Silk Only, pretty:SSDACLOGO_190X190, symbol xSSDAC:SSDAC_LOGO
Other:
- added sheet Color LEDs (RGB_LEDs.kicad_sch)
- sheet SerialDAC: file Serialdac-dff.kicad_sch -> Serialdac.kicad_sch
- company: xken -> Xken
- title: xSSDAC SD player v1.1  -> xSSDAC SD player v2.0
Changed lines of the file:
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@@
   (paper "A4")
   (title_block
-    (title "xSSDAC SD player v1.1 ")
+    (title "xSSDAC SD player v2.0")
     (date "2023-06-24")
-    (company "xken")
+    (company "Xken")
   )
   (symbol (lib_id "Mechanical:MountingHole_Pad") (at 163.83 88.9 0) (unit 1)
@@
     )
     (property "Datasheet" "~" (at 163.83 88.9 0)
+      (effects (font (size 1.27 1.27)) hide)
+    )
+    (property "Akizuki Price/Stock" "" (at 163.83 88.9 0)
+      (effects (font (size 1.27 1.27)) hide)
+    )
+    (property "Description" "Mounting hole with electrical contact 2.7mm" (at 163.83 88.9 0)
+      (effects (font (size 1.27 1.27)) hide)
+    )
+    (property "Akizuki Part Number" "" (at 163.83 88.9 0)
       (effects (font (size 1.27 1.27)) hide)
     )
@@
       (effects (font (size 1.27 1.27)) hide)
     )
+    (property "Akizuki Price/Stock" "" (at 163.83 118.11 0)
+      (effects (font (size 1.27 1.27)) hide)
+    )
+    (property "Description" "Mounting hole with electrical contact 2.7mm" (at 163.83 118.11 0)
+      (effects (font (size 1.27 1.27)) hide)
+    )
+    (property "Akizuki Part Number" "" (at 163.83 118.11 0)
+      (effects (font (size 1.27 1.27)) hide)
+    )
     (pin "1")
     (instances
@@
       (effects (font (size 1.27 1.27)) hide)
     )
+    (property "Akizuki Price/Stock" "" (at 198.12 88.9 0)
+      (effects (font (size 1.27 1.27)) hide)
+    )
+    (property "Description" "Mounting hole with electrical contact 2.7mm" (at 198.12 88.9 0)
+      (effects (font (size 1.27 1.27)) hide)
+    )
+    (property "Akizuki Part Number" "" (at 198.12 88.9 0)
+      (effects (font (size 1.27 1.27)) hide)
+    )
     (pin "1")
     (instances
@@
       (effects (font (size 1.27 1.27)) hide)
     )
+    (property "Akizuki Price/Stock" "" (at 198.12 118.11 0)
+      (effects (font (size 1.27 1.27)) hide)
+    )
+    (property "Description" "Mounting hole with electrical contact 2.7mm" (at 198.12 118.11 0)
+      (effects (font (size 1.27 1.27)) hide)
+    )
+    (property "Akizuki Part Number" "" (at 198.12 118.11 0)
+      (effects (font (size 1.27 1.27)) hide)
+    )
     (pin "1")
     (instances
@@
       (effects (font (size 1.27 1.27)) hide)
     )
+    (property "Akizuki Price/Stock" "" (at 163.83 93.98 0)
+      (effects (font (size 1.27 1.27)) hide)
+    )
+    (property "Akizuki Part Number" "" (at 163.83 93.98 0)
+      (effects (font (size 1.27 1.27)) hide)
+    )
     (pin "1")
     (pin "2")
@@
       (effects (font (size 1.27 1.27)) hide)
     )
+    (property "Akizuki Price/Stock" "" (at 198.12 93.98 0)
+      (effects (font (size 1.27 1.27)) hide)
+    )
+    (property "Akizuki Part Number" "" (at 198.12 93.98 0)
+      (effects (font (size 1.27 1.27)) hide)
+    )
     (pin "1")
     (pin "2")
@@
       (effects (font (size 1.27 1.27)) hide)
     )
+    (property "Akizuki Price/Stock" "" (at 163.83 123.19 0)
+      (effects (font (size 1.27 1.27)) hide)
+    )
+    (property "Akizuki Part Number" "" (at 163.83 123.19 0)
+      (effects (font (size 1.27 1.27)) hide)
+    )
     (pin "1")
     (pin "2")
@@
     )
     (property "Datasheet" "~" (at 198.12 123.19 0)
+      (effects (font (size 1.27 1.27)) hide)
+    )
+    (property "Akizuki Price/Stock" "" (at 198.12 123.19 0)
+      (effects (font (size 1.27 1.27)) hide)
+    )
+    (property "Akizuki Part Number" "" (at 198.12 123.19 0)
       (effects (font (size 1.27 1.27)) hide)
     )
@@
     )
   )
-  (sheet (at 24.13 25.4) (size 54.61 39.37) (fields_autoplaced)
+  (symbol (lib_id "xSSDAC:Logo_SSDAC") (at 231.14 149.86 0) (unit 1)
+    (in_bom no) (on_board no) (dnp no) (fields_autoplaced)
+    (property "Reference" "#SYM2" (at 231.14 144.78 0)
+      (effects (font (size 1.27 1.27)) hide)
+    )
+    (property "Value" "Logo_SSDAC" (at 231.14 152.4 0)
+      (effects (font (size 1.27 1.27)) hide)
+    )
+    (property "Footprint" "" (at 231.14 149.86 0)
+      (effects (font (size 1.27 1.27)) hide)
+    )
+    (property "Datasheet" "SSDAC" (at 231.14 149.86 0)
+      (effects (font (size 1.27 1.27)) hide)
+    )
+    (property "Sim.Enable" "0" (at 231.14 147.32 0)
+      (effects (font (size 1.27 1.27)) hide)
+    )
+    (instances
+      (project "xSSDAC"
+        (path "/55bc7a0a-7b3c-4fcf-be7b-a0c136882cfb"
+          (reference "#SYM2") (unit 1)
+        )
+      )
+    )
+  )
+  (symbol (lib_id "xSSDAC:SSDAC_LOGO") (at 40.64 144.78 0) (unit 1)
+    (in_bom yes) (on_board yes) (dnp no)
+    (property "Reference" "ART1" (at 36.83 139.7 0)
+      (effects (font (size 2 2)) (justify left))
+    )
+    (property "Value" "Silk Only" (at 40.64 144.78 0) (show_name)
+      (effects (font (size 1.27 1.27)))
+    )
+    (property "Footprint" "pretty:SSDACLOGO_190X190" (at 52.07 147.32 0) (show_name)
+      (effects (font (size 1.27 1.27)))
+    )
+    (property "Datasheet" "" (at 40.64 144.78 0)
+      (effects (font (size 1.27 1.27)) hide)
+    )
+    (property "Akizuki Price/Stock" "" (at 40.64 144.78 0)
+      (effects (font (size 1.27 1.27)) hide)
+    )
+    (property "Description" "SSDAC logo mark" (at 40.64 144.78 0)
+      (effects (font (size 1.27 1.27)) hide)
+    )
+    (property "Akizuki Part Number" "" (at 40.64 144.78 0)
+      (effects (font (size 1.27 1.27)) hide)
+    )
+    (instances
+      (project "xSSDAC"
+        (path "/55bc7a0a-7b3c-4fcf-be7b-a0c136882cfb"
+          (reference "ART1") (unit 1)
+        )
+      )
+    )
+  )
+  (symbol (lib_id "xSSDAC:Logo_SSDAC") (at -36.83 135.89 0) (unit 1)
+    (in_bom no) (on_board no) (dnp no) (fields_autoplaced)
+    (property "Reference" "#SYM1" (at -36.83 130.81 0)
+      (effects (font (size 1.27 1.27)) hide)
+    )
+    (property "Value" "Logo_SSDAC" (at -36.83 138.43 0)
+      (effects (font (size 1.27 1.27)) hide)
+    )
+    (property "Footprint" "" (at -36.83 135.89 0)
+      (effects (font (size 1.27 1.27)) hide)
+    )
+    (property "Datasheet" "SSDAC" (at -36.83 135.89 0)
+      (effects (font (size 1.27 1.27)) hide)
+    )
+    (property "Sim.Enable" "0" (at -36.83 133.35 0)
+      (effects (font (size 1.27 1.27)) hide)
+    )
+    (instances
+      (project "xSSDAC"
+        (path "/55bc7a0a-7b3c-4fcf-be7b-a0c136882cfb"
+          (reference "#SYM1") (unit 1)
+        )
+      )
+    )
+  )
+  (sheet (at 24.13 25.4) (size 54.61 27.94) (fields_autoplaced)
     (stroke (width 0) (type solid))
     (fill (color 0 0 0 0.0000))
@@
       (effects (font (size 1.27 1.27)) (justify left bottom))
     )
-    (property "Sheetfile" "xCORE.kicad_sch" (at 24.13 65.3546 0)
+    (property "Sheetfile" "xCORE.kicad_sch" (at 24.13 53.9246 0)
       (effects (font (size 1.27 1.27)) (justify left top))
     )
@@
     )
   )
-  (sheet (at 88.9 25.4) (size 54.61 39.37) (fields_autoplaced)
+  (sheet (at 88.9 25.4) (size 54.61 27.94) (fields_autoplaced)
     (stroke (width 0) (type solid))
     (fill (color 0 0 0 0.0000))
@@
       (effects (font (size 1.27 1.27)) (justify left bottom))
     )
-    (property "Sheetfile" "Serialdac-dff.kicad_sch" (at 88.9 65.3546 0)
+    (property "Sheetfile" "Serialdac.kicad_sch" (at 88.9 53.9246 0)
       (effects (font (size 1.27 1.27)) (justify left top))
     )
@@
     )
   )
-  (sheet (at 154.94 25.4) (size 54.61 39.37) (fields_autoplaced)
+  (sheet (at 154.94 25.4) (size 54.61 27.94) (fields_autoplaced)
     (stroke (width 0) (type solid))
     (fill (color 0 0 0 0.0000))
@@
       (effects (font (size 1.27 1.27)) (justify left bottom))
     )
-    (property "Sheetfile" "SDcard.kicad_sch" (at 154.94 65.3546 0)
+    (property "Sheetfile" "SDcard.kicad_sch" (at 154.94 53.9246 0)
       (effects (font (size 1.27 1.27)) (justify left top))
     )
@@
     )
   )
-  (sheet (at 24.13 80.01) (size 54.61 41.91) (fields_autoplaced)
+  (sheet (at 24.13 80.01) (size 54.61 27.94) (fields_autoplaced)
     (stroke (width 0) (type solid))
     (fill (color 0 0 0 0.0000))
@@
       (effects (font (size 1.27 1.27)) (justify left bottom))
     )
-    (property "Sheetfile" "UnusedPin.kicad_sch" (at 24.13 122.5046 0)
+    (property "Sheetfile" "UnusedPin.kicad_sch" (at 24.13 108.5346 0)
       (effects (font (size 1.27 1.27)) (justify left top))
     )
@@
       )
     )
+  )
+  (sheet (at 88.9 80.01) (size 54.61 27.94) (fields_autoplaced)
+    (stroke (width 0.1524) (type solid))
+    (fill (color 0 0 0 0.0000))
+    (property "Sheetname" "Color LEDs" (at 88.9 79.2984 0)
+      (effects (font (size 1.27 1.27)) (justify left bottom))
+    )
+    (property "Sheetfile" "RGB_LEDs.kicad_sch" (at 88.9 108.5346 0)
+      (effects (font (size 1.27 1.27)) (justify left top))
+    )
+    (instances
+      (project "xSSDAC"
+        (path "/55bc7a0a-7b3c-4fcf-be7b-a0c136882cfb" (page "6"))
+      )
+    )
